File: RP2040_minimal.kicad_sch (KiCad schematic)
At the start: 34 parts, among them J1 Conn_02x18_Odd_Even, J2 Conn_01x02, J3 USB_B_Micro, J4 Conn_02x18_Odd_Even, U1 NCP1117-3.3_SOT223, U2 W25Q128JVS, U3 RP2040, Y1 ABLS-12.000MHZ-B4-T

Commit message: prepare fabrication outputs
Parts:
- C1, C17, C2: LCSC (none) -> C15850
- C10, C12, C13, C16, C3, C4, C5, C6, C7, C8: LCSC (none) -> C126504
- C11, C9: LCSC (none) -> C307331
- C14, C15: LCSC (none) -> C52923
- J1, J4: LCSC (none) -> C168945
- J2: LCSC (none) -> C124375
- J3: LCSC (none) -> C428495
- R2, R5: LCSC (none) -> C11702
- R3, R4: LCSC (none) -> C274349
- U1: LCSC (none) -> C26537
- U2: LCSC (none) -> C97521
- U3: LCSC (none) -> C2040
- Y1: LCSC (none) -> C110563
